File: projekt.kicad_sch (KiCad schematic)
At the start: 23 parts, among them IC1 DW01+G, J1 USB_C_Receptacle_PowerOnly_24P, J2 TP4056, J3 Conn_01x04_Pin, U1 ESP32-WROOM-32D, U4 TB6612FNG, U5 MPU-6050, U7 AMS1117-3.3

Commit message: Prawie skończony schemat.
Parts:
- added C10, C5, C6, C7, C8, C9: 0.1u, symbol Device:C
- added C11: 10u, symbol Device:C
- added C12, C13: 100n, symbol Device:C
- added J4: Conn_01x02_Socket, Connector_JST:JST_XH_B2B-XH-A_1x02_P2.50mm_Vertical, symbol Connector:Conn_01x02_Socket
- added J5: AO1, symbol Connector:Conn_01x01_Pin
- added J6: AO2, symbol Connector:Conn_01x01_Pin
- added J7: BO1, symbol Connector:Conn_01x01_Pin
- added J8: BO2, symbol Connector:Conn_01x01_Pin
- added Q1, Q2: AO3400A, Package_TO_SOT_SMD:SOT-23, symbol Transistor_FET:AO3400A
- added R10: 10k, symbol Device:R
- added R8: 100, symbol Device:R
- added R9: 1k, symbol Device:R
- R5: value R -> 43k
- R6: value R -> 180k
- TH1: value 10k -> 100k
Connections:
- net +3.3V: now also C6.1, R10.1
- net GND: now also U1.1 (GND), U1.15 (GND), U1.38 (GND), U1.39 (GND), U4.10 (PGND2), U4.18 (GND), U4.3 (PGND1), U4.4 (PGND1), U4.9 (PGND2), U5.1 (CLKIN), U5.11 (FSYNC), U5.18 (GND), C10.2, C11.2, C12.2, C13.2, C6.2, C7.2, C8.2, C9.2, Q2.2 (S), R9.1
- net LIPO+: now also U4.13 (VM2), U4.14 (VM3), U4.24 (VM1), C10.1, C11.1, C8.1, C9.1, J4.1 (Pin_1), R8.1
- net RX: now also U1.35 (TXD0/IO1)
- net TX: now also U1.34 (RXD0/IO3)
- net +3V3: now reaches U5.13 (VDD)
- net +3V3: now also U4.20 (VCC), U5.8 (VLOGIC), C12.1, C13.1, C7.1
- net IO26: now reaches U1.11 (IO26)
- net IO26: now also U4.17 (BIN1)
- net IO27: now reaches U1.12 (IO27)
- net IO27: now also U4.16 (BIN2)
- net IO17: now reaches U1.28 (IO17)
- net at U1.3 (EN): now also R10.2
- net IO18: now reaches U1.30 (IO18)
- net IO18: now also U4.15 (PWMB), U4.19 (STBY)
- net IO19: now reaches U1.31 (IO19)
- net IO19: now also U4.23 (PWMA)
- net IO22: now reaches U1.36 (IO22)
- net IO22: now also U4.21 (AIN1)
- net IO23: now reaches U1.37 (IO23)
- net IO23: now also U4.22 (AIN2)
- net at IC1.1 (OD): now also Q1.1 (G)
- net at IC1.2 (CS): now also R9.2
- net at IC1.3 (OC): now also Q2.1 (G)
- net at IC1.5 (VCC): now also C5.2, R8.2
- net LIPO-: now reaches IC1.6 (GND)
- net LIPO-: now also C5.1, J4.2 (Pin_2), Q1.2 (S)
- net at U4.1 (AO1), U4.2 (AO1): now also J5.1 (Pin_1)
- net at U4.11 (BO1), U4.12 (BO1): now also J7.1 (Pin_1)
- net at U4.5 (AO2), U4.6 (AO2): now also J6.1 (Pin_1)
- net at U4.7 (BO2), U4.8 (BO2): now also J8.1 (Pin_1)
- new net: Q1.3 (D), Q2.3 (D)
- no-connect marks 0 -> 2
Other:
- note added: "MPU"
- note added: "Sterownik silników"
- note added: "Tu podłączone do GND, żeby układ zabezpieczeń tym sterował."
- note added: "Układ zabezpieczeń"
- note added: "Układ ładowania baterii"
- note added: "Wejście programatora"
- moved on the sheet: C2, C3, D1, IC1, U4, U5, U7

Commit message: Prawie skończony schemat
Parts:
- removed U1: ESP32-WROOM-32D, RF_Module:ESP32-WROOM-32D, symbol RF_Module:ESP32-WROOM-32D
- removed U5: MPU-6050, Sensor_Motion:InvenSense_QFN-24_4x4mm_P0.5mm, symbol Sensor_Motion:MPU-6050
- added AC1: ADXL345, CC-14-1, symbol SamacSys_Parts:ADXL345
- added D4, D5: WHITE, LED_SMD:LED_0603_1608Metric_Pad1.05x0.95mm_HandSolder, symbol Device:LED
- added D6, D7: RED, LED_SMD:LED_0603_1608Metric_Pad1.05x0.95mm_HandSolder, symbol Device:LED
- added Q3, Q4, Q5, Q6: AO3400A, Package_TO_SOT_SMD:SOT-23, symbol Transistor_FET:AO3400A
- added R11, R12: 4.7k, symbol Device:R
- added R13, R14, R15, R16: 1k, Resistor_SMD:R_0603_1608Metric_Pad0.98x0.95mm_HandSolder, symbol Device:R
- added SW2: SW_DPDT_x2, symbol Switch:SW_DPDT_x2
- added TP1: BOOT PIN, symbol Connector:TestPoint
- added TP2: TDI, symbol Connector:TestPoint
- added TP3: TCK, symbol Connector:TestPoint
- added TP4: TMS, symbol Connector:TestPoint
- added TP5: TDO, symbol Connector:TestPoint
- added U2: ESP32-WROOM-32E, RF_Module:ESP32-WROOM-32D, symbol RF_Module:ESP32-WROOM-32E
Connections:
- net +3.3V: now also U2.2 (VDD)
- net +3V3: now also AC1.1 (VDD_I/O), AC1.6 (VS), AC1.7 (~{CS}), Q3.2 (S), Q4.2 (S), Q5.2 (S), Q6.2 (S)
- net GND: now also AC1.12 (SDO/ALT_ADDRESS), AC1.2 (GND_1), AC1.4 (GND_2), AC1.5 (GND_3), R11.1, R12.2, R13.2, R14.2, R15.2, R16.2, U2.1 (GND), U2.15 (GND), U2.38 (GND), U2.39 (GND)
- net IO17: now also U2.28 (IO17)
- net IO18: now also U2.30 (IO18)
- net IO19: now also U2.31 (IO19)
- net IO22: now also U2.36 (IO22)
- net IO23: now also U2.37 (IO23)
- net IO26: now also U2.11 (IO26)
- net IO27: now also U2.12 (IO27)
- net LIPO+: now also SW2.2 (B); no longer C10.1, C11.1, C2.1, C8.1, C9.1, D1.1 (K), U4.13 (VM2), U4.14 (VM3), U4.24 (VM1), U7.3 (VI)
- net RX: now also U2.35 (TXD0/IO1)
- net TX: now also U2.34 (RXD0/IO3)
- net at R10.2: now also U2.3 (EN)
- new net: D4.1 (K), R13.1
- new net: D4.2 (A), Q3.3 (D)
- new net: TP4.1, U2.13 (IO14)
- new net: TP2.1, U2.14 (IO12)
- new net: TP3.1, U2.16 (IO13)
- new net: TP5.1, U2.23 (IO15)
- new net: TP1.1, U2.25 (IO0)
- new net: D5.1 (K), R14.1
- new net: D5.2 (A), Q4.3 (D)
- new net: D7.1 (K), R16.1
- new net: D7.2 (A), Q6.3 (D)
- new net: D6.1 (K), R15.1
- new net: D6.2 (A), Q5.3 (D)
- new net ACC_IT1: AC1.9 (INT2), U2.6 (IO34)
- new net ACC_IT2: AC1.8 (INT1), U2.7 (IO35)
- new net ACC_SCL: AC1.14 (SCL/SCLK), R12.1, U2.26 (IO4)
- new net ACC_SDA: AC1.13 (SDA/SDI/SDIO), R11.2, U2.27 (IO16)
- new net LED1: Q3.1 (G), U2.24 (IO2)
- new net LED2: Q4.1 (G), U2.29 (IO5)
- new net LED3: Q5.1 (G), U2.8 (IO32)
- new net LED4: Q6.1 (G), U2.9 (IO33)
- new net PWR+: C10.1, C11.1, C2.1, C8.1, C9.1, D1.1 (K), SW2.1 (A), U4.13 (VM2), U4.14 (VM3), U4.24 (VM1), U7.3 (VI)
- no-connect marks 2 -> 8
Other:
- note added: "Akcelerometr"
- note added: "Biała"
- note added: "Czerwona"
- note added: "Diody LED"
- note added: "To jest ok?"
- note added: "Wejście baterii i przełącznik"
- note added: "Wyjścia dla potencjalnego programatora JTAG"
- company: (none) -> Igor Santarek, Kamil Lewiński
- title: (none) -> Mini RC Car
- moved on the sheet: C12, C13, C2, C3, D1, J4, U7

Commit message: Potwarz dla ludzkości
Parts:
- removed SW2: SW_DPDT_x2, symbol Switch:SW_DPDT_x2
- added Q7: IRLML6344TRPBF, SOT95P237X112-3N, symbol SamacSys_Parts:IRLML6344TRPBF
- added R17, R19, R20, R23: 10, Resistor_SMD:R_0603_1608Metric_Pad0.98x0.95mm_HandSolder, symbol Device:R
- added R18, R22: 10k, Resistor_SMD:R_0603_1608Metric_Pad0.98x0.95mm_HandSolder, symbol Device:R
- added R21, R24: 100, Resistor_SMD:R_0603_1608Metric_Pad0.98x0.95mm_HandSolder, symbol Device:R
- added R25: 10, symbol Device:R
- added R26: 10k, symbol Device:R
- added SW1: SW_Slide_DPDT, Button_Switch_THT:SW_CK_JS202011AQN_DPDT_Angled, symbol Switch:SW_Slide_DPDT
- R13, R16: value 1k -> 10
- R14, R15: value 1k -> 10k
- R3, R4: value 1k -> 130
Connections:
- net PWR+ is gone; now on net LIPO+: C10.1, C11.1, C2.1, C8.1, C9.1, D1.1 (K), U4.13 (VM2), U4.14 (VM3), U4.24 (VM1), U7.3 (VI)
- net +3V3: now also R11.1, R12.2, R13.2, R20.2, R21.2, R24.2; no longer Q3.2 (S), Q4.2 (S), Q5.2 (S), Q6.2 (S)
- net LED1: now also R17.2; no longer Q3.1 (G)
- net LED2: now also R16.2; no longer Q4.1 (G)
- net LED3: now also R23.2; no longer Q5.1 (G)
- net LED4: now also R19.2; no longer Q6.1 (G)
- net LIPO+: now also SW1.2 (B), SW1.5 (B)
- net at D4.1 (K): now also Q3.3 (D); no longer R13.1
- net at D4.2 (A): now also R13.1; no longer Q3.3 (D)
- net at D5.1 (K): now also Q4.3 (D); no longer R14.1
- net at D5.2 (A): now also R20.1; no longer Q4.3 (D)
- net at R16.1: now also Q5.1 (G), R15.2; no longer D7.1 (K)
- net at Q6.3 (D): now also D7.1 (K); no longer D7.2 (A)
- net at D6.1 (K): now also Q5.3 (D); no longer R15.1
- net at D6.2 (A): now also R21.1; no longer Q5.3 (D)
- net GND renamed GND2
- net GND2: now also Q7.3 (D); no longer C1.1, C4.2, J1.A1 (GND), J1.A12 (GND), J1.B1 (GND), J1.B12 (GND), J1.S1 (SHIELD), J2.3 (GND_3), J2.9 (EP), J3.3 (Pin_3), Q2.2 (S), R1.2, R11.1, R12.2, R13.2, R14.2, R15.2, R16.2, R2.2, R6.2, R7.1, R9.1, TH1.1
- new net: Q4.1 (G), R14.2, R19.1
- new net: Q3.1 (G), R17.1, R18.2
- new net: Q6.1 (G), R22.2, R23.1
- new net: Q7.1 (G), R25.2, R26.1
- new net: D7.2 (A), R24.1
- new net GND1: C1.1, C4.2, J1.A1 (GND), J1.A12 (GND), J1.B1 (GND), J1.B12 (GND), J1.S1 (SHIELD), J2.3 (GND_3), J2.9 (EP), J3.3 (Pin_3), Q2.2 (S), Q3.2 (S), Q4.2 (S), Q5.2 (S), Q6.2 (S), Q7.2 (S), R1.2, R14.1, R15.1, R18.1, R2.2, R22.1, R26.2, R6.2, R7.1, R9.1, TH1.1
- new net SW+: R25.1, SW1.1 (A), SW1.6 (C)
- no-connect marks 8 -> 7
Other:
- note added: "BRUH??"
- note removed: "To jest ok?"
- moved on the sheet: C1, C2, C3, D1, D4, Q3, R13, U7

Commit message: Gotowy schemat (albo prawie gotowy)
Parts:
- removed J5: AO1, symbol Connector:Conn_01x01_Pin
- removed J6: AO2, symbol Connector:Conn_01x01_Pin
- removed J7: BO1, symbol Connector:Conn_01x01_Pin
- removed J8: BO2, symbol Connector:Conn_01x01_Pin
- removed Q7: IRLML6344TRPBF, SOT95P237X112-3N, symbol SamacSys_Parts:IRLML6344TRPBF
- removed TP1: BOOT PIN, symbol Connector:TestPoint
- added C14: 10u, Capacitor_SMD:C_0603_1608Metric_Pad1.08x0.95mm_HandSolder, symbol Device:C
- added C15: 10n, Capacitor_SMD:C_0603_1608Metric_Pad1.08x0.95mm_HandSolder, symbol Device:C
- added C16: 1u, Capacitor_SMD:C_0603_1608Metric_Pad1.08x0.95mm_HandSolder, symbol Device:C
- added C17: 100n, Capacitor_SMD:C_0603_1608Metric_Pad1.08x0.95mm_HandSolder, symbol Device:C
- added D8: GREEN, LED_SMD:LED_0805_2012Metric_Pad1.15x1.40mm_HandSolder, symbol Device:LED
- added J10: BO1, symbol Connector:Conn_01x02_Socket
- added J5: AO2, symbol Connector:Conn_01x02_Socket
- added J6: BO2, symbol Connector:Conn_01x02_Socket
- added J9: AO1, symbol Connector:Conn_01x02_Socket
- added R27: 1k, Resistor_SMD:R_0603_1608Metric_Pad0.98x0.95mm_HandSolder, symbol Device:R
- added S1: AP22800HB-7, SON50P161X211X60-9N, symbol SamacSys_Parts:AP22800HB-7
- added SW2: RST, symbol Switch:SW_Push
- added SW3: BOOT, symbol Switch:SW_Push
- C10, C6, C8, C9: value 0.1u -> 100n; footprint (none) -> Capacitor_SMD:C_0603_1608Metric_Pad1.08x0.95mm_HandSolder
- C11, C12, C13, C5, C7: footprint (none) -> Capacitor_SMD:C_0603_1608Metric_Pad1.08x0.95mm_HandSolder
- D1: footprint (none) -> Diode_SMD:D_0603_1608Metric_Pad1.05x0.95mm_HandSolder
- D2, D3: footprint (none) -> LED_SMD:LED_0805_2012Metric_Pad1.15x1.40mm_HandSolder
- D4, D5, D6, D7: footprint LED_SMD:LED_0603_1608Metric_Pad1.05x0.95mm_HandSolder -> LED_SMD:LED_0805_2012Metric_Pad1.15x1.40mm_HandSolder
- J1: footprint (none) -> Connector_USB:USB_C_Receptacle_GCT_USB4125-xx-x-0190_6P_TopMnt_Horizontal
- J3: footprint (none) -> Connector_PinHeader_2.54mm:PinHeader_1x04_P2.54mm_Vertical
- R10, R11, R12, R8, R9: footprint (none) -> Resistor_SMD:R_0603_1608Metric_Pad0.98x0.95mm_HandSolder
- R13, R20: value 10 -> 60
- R16, R17, R19, R23: value 10 -> 330
- R21, R24: value 100 -> 260
- R25: value 10 -> 4.7k; footprint (none) -> Resistor_SMD:R_0603_1608Metric_Pad0.98x0.95mm_HandSolder
- R26: value 10k -> 100; footprint (none) -> Resistor_SMD:R_0603_1608Metric_Pad0.98x0.95mm_HandSolder
- R3, R4: value 130 -> 1k
Connections:
- net GND2 is gone; now on net GND: AC1.12 (SDO/ALT_ADDRESS), AC1.2 (GND_1), AC1.4 (GND_2), AC1.5 (GND_3), C10.2, C11.2, C12.2, C13.2, C2.2, C3.2, C6.2, C7.2, C8.2, C9.2, U2.1 (GND), U2.15 (GND), U2.38 (GND), U2.39 (GND), U4.10 (PGND2), U4.18 (GND), U4.3 (PGND1), U4.4 (PGND1), U4.9 (PGND2), U7.1 (GND)
- net +3.3V: now also R10.2; no longer R10.1
- net LED1: now also R18.2
- net LED2: now also R15.2
- net LED3: now also R22.2
- net LED4: now also R14.2
- net LIPO+: now also C14.2, S1.1 (VIN_1), S1.2 (VIN_2); no longer C10.1, C11.1, C2.1, C8.1, C9.1, D1.1 (K), U4.13 (VM2), U4.14 (VM3), U4.24 (VM1), U7.3 (VI)
- net RX: now also J3.2 (Pin_2); no longer J3.1 (Pin_1)
- net SW+: now also R25.2, S1.3 (EN); no longer R25.1
- net TX: now also J3.3 (Pin_3); no longer J3.2 (Pin_2)
- net at Q4.1 (G), R19.1: no longer R14.2
- net at U4.11 (BO1), U4.12 (BO1): now also J10.1 (Pin_1), J10.2 (Pin_2)
- net at U2.25 (IO0): now also SW3.2
- net at U2.3 (EN): now also R10.1, C17.1, SW2.2; no longer R10.2
- net at Q3.1 (G), R17.1: no longer R18.2
- net at U4.1 (AO1), U4.2 (AO1): now also J9.1 (Pin_1), J9.2 (Pin_2)
- net at Q6.1 (G), R23.1: no longer R22.2
- net at R26.1: now also S1.6 (DIS); no longer R25.2
- net at Q5.1 (G), R16.1: no longer R15.2
- net at U4.5 (AO2), U4.6 (AO2): now also J5.1 (Pin_1), J5.2 (Pin_2)
- net at U4.7 (BO2), U4.8 (BO2): now also J6.1 (Pin_1), J6.2 (Pin_2)
- net GND1 renamed GND
- net GND: now also J3.1 (Pin_1), R25.1, C14.1, C15.1, C16.2, C17.2, D8.1 (K), S1.9 (GND), SW2.1, SW3.1; no longer J3.3 (Pin_3), R26.2
- new net: C15.2, S1.4 (SS)
- new net: D8.2 (A), R27.1, S1.5 (PG)
- new net PWR+: C10.1, C11.1, C16.1, C2.1, C8.1, C9.1, D1.1 (K), R26.2, R27.2, S1.7 (VOUT_1), S1.8 (VOUT_2), U4.13 (VM2), U4.14 (VM3), U4.24 (VM1), U7.3 (VI)
- no-connect marks 7 -> 8
Other:
- note removed: "BRUH??"
- note removed: "Wejście baterii i przełącznik"
- moved on the sheet: C2, C3, C7, D1, J4, R10, SW1, U7

Commit message: Poprawienie footprintów i ustawień
Parts:
- removed AC1: ADXL345, CC-14-1, symbol SamacSys_Parts:ADXL345
- removed J1: USB_C_Receptacle_PowerOnly_24P, Connector_USB:USB_C_Receptacle_GCT_USB4125-xx-x-0190_6P_TopMnt_Horizontal, symbol Connector:USB_C_Receptacle_PowerOnly_24P
- removed J10: BO1, symbol Connector:Conn_01x02_Socket
- removed J5: AO2, symbol Connector:Conn_01x02_Socket
- removed J6: BO2, symbol Connector:Conn_01x02_Socket
- removed J9: AO1, symbol Connector:Conn_01x02_Socket
- added AC2: ADXL345, CC-14-1, symbol SamacSys_Parts:ADXL345
- added J11, J5: AO1, TestPoint:TestPoint_Pad_2.0x2.0mm, symbol Connector:Conn_01x01_Socket
- added J12, J9: BO2, TestPoint:TestPoint_Pad_2.0x2.0mm, symbol Connector:Conn_01x01_Socket
- added J13, J14: BO1, TestPoint:TestPoint_Pad_2.0x2.0mm, symbol Connector:Conn_01x01_Socket
- added J6: USB_C_Receptacle_PowerOnly_6P, Connector_USB:USB_C_Receptacle_GCT_USB4125-xx-x-0190_6P_TopMnt_Horizontal, symbol Connector:USB_C_Receptacle_PowerOnly_6P
- added J7, J8: AO2, TestPoint:TestPoint_Pad_2.0x2.0mm, symbol Connector:Conn_01x01_Socket
- SW2, SW3: footprint (none) -> Button_Switch_SMD:SW_Push_1P1T_NO_CK_KSC7xxJ
- TP2, TP3, TP4, TP5: footprint (none) -> TestPoint:TestPoint_Pad_2.0x2.0mm
Connections:
- net +3V3: now also AC2.1 (VDD_I/O), AC2.6 (VS), AC2.7 (~{CS})
- net ACC_IT1: now also AC2.9 (INT2)
- net ACC_IT2: now also AC2.8 (INT1)
- net ACC_SCL: now also AC2.14 (SCL/SCLK)
- net ACC_SDA: now also AC2.13 (SDA/SDI/SDIO)
- net GND: now also AC2.12 (SDO/ALT_ADDRESS), AC2.2 (GND_1), AC2.4 (GND_2), AC2.5 (GND_3), J6.A12 (GND), J6.B12 (GND), J6.S1 (SHIELD)
- net VCC: now also J6.A9 (VBUS), J6.B9 (VBUS)
- net at U4.7 (BO2), U4.8 (BO2): now also J12.1 (Pin_1), J9.1 (Pin_1)
- net at R2.1: now also J6.A5 (CC1)
- net at U4.1 (AO1), U4.2 (AO1): now also J11.1 (Pin_1), J5.1 (Pin_1)
- net at U4.5 (AO2), U4.6 (AO2): now also J7.1 (Pin_1), J8.1 (Pin_1)
- net at R1.1: now also J6.B5 (CC2)
- net at U4.11 (BO1), U4.12 (BO1): now also J13.1 (Pin_1), J14.1 (Pin_1)
