File: projekt.kicad_sch (KiCad schematic)
At the start: 95 parts, among them IC1 DW01+G, IC2 SS8050-HF, IC3 SS8050-HF, J1 CO1, J10 Conn_01x06_Pin, J11 AO1, J12 BO2, J14 BO1, J2 TP4056, J4 Conn_01x02_Socket, J5 CO2, J6 USB_C_Receptacle_PowerOnly_24P, J7 DO1, J8 AO2, J9 DO2, Q1 AO3400A, Q2 AO3400A, Q3 AO3400A, Q4 AO3400A, Q5 AO3400A, Q6 AO3400A, SW1 SW_Slide_DPDT, SW2 RST, SW3 BOOT, U1 TB6612FNG, U2 ESP32-WROOM-32E, U4 TB6612FNG, U7 AMS1117-3.3

Commit message: Poprawienie schematu i PCB
Parts:
- removed D1: D, Diode_SMD:D_0603_1608Metric_Pad1.05x0.95mm_HandSolder, symbol Device:D
- removed IC2, IC3: SS8050-HF, SOT95P240X115-3N, symbol SamacSys_Parts:SS8050-HF
- removed R22: 10k, Resistor_SMD:R_0603_1608Metric_Pad0.98x0.95mm_HandSolder, symbol Device:R
- removed U7: AMS1117-3.3, Package_TO_SOT_SMD:SOT-223-3_TabPin2, symbol Regulator_Linear:AMS1117-3.3
- added IC4: MIC5504-3.3YM5-TR, SOT95P280X145-5N, symbol SamacSys_Parts:MIC5504-3.3YM5-TR
- added Q7, Q8: SS8050-HF, SOT95P240X115-3N, symbol Simulation_SPICE:NPN
- C3: value 4.7u -> 1u
- R13, R20: value 60 -> 120
- R21, R24: value 260 -> 320
- renumbered J11 to AO1, J8 to AO2, J14 to BO1, J12 to BO2, J1 to CO1, J5 to CO2, J7 to DO1, J9 to DO2
Connections:
- net +3.3V: now also IC4.5 (VOUT)
- net +3V3: no longer R13.2, R20.2, R21.2, R24.2
- net BOOT: now also U1.19 (STBY), U4.19 (STBY), Q8.1 (C)
- net DTR: now also Q8.3 (E)
- net EN: now also Q7.1 (C)
- net GND: now also IC4.2 (GND)
- net IO12: no longer U1.23 (PWMA), U2.14 (IO12)
- net IO15: no longer U1.16 (BIN2), U2.23 (IO15)
- net LED3: now also U2.23 (IO15); no longer U2.8 (IO32)
- net LIPO+: now also C2.1, IC4.1 (VIN)
- net PWR+: now also R13.2, R20.2, R21.2, R24.2; no longer C2.1
- net RTS: now also Q7.3 (E)
- net SW+: now also IC4.3 (EN)
- net at R28.1: now also Q8.2 (B)
- net at R15.1: now also Q7.2 (B)
- net IO13 renamed PWMD
- net IO14 renamed DIN1
- net IO18 renamed PWMB
- net PWMB: no longer U1.19 (STBY), U4.19 (STBY)
- net IO19 renamed PWMA
- net IO21 renamed CIN1
- net IO22 renamed AIN1
- net IO23 renamed AIN2
- net IO25 renamed CIN2
- net IO26 renamed BIN1
- net IO27 renamed BIN2
- new net DIN2: U1.16 (BIN2), U2.8 (IO32)
- new net PWMC: U1.23 (PWMA), U2.14 (IO12)
- no-connect marks 6 -> 7
Other:
- moved on the sheet: C1, C16, C2, C3, D8, J6, R1, R2, R26, R27, R7

Commit message: powoli nabiera koloru
Parts:
- TH1: footprint Resistor_SMD:R_0603_1608Metric_Pad0.98x0.95mm_HandSolder -> Resistor_SMD:Termistor_SMD
Connections:
- net +3V3 is gone; now on net +3.3V: AC2.1 (VDD_I/O), AC2.6 (VS), AC2.7 (~{CS}), C12.1, C13.1, C18.1, C23.1, C24.1, C7.1, R11.1, R12.2, U1.20 (VCC), U4.20 (VCC)
- net IO12 is gone; now on net PWMC: R30.2
- net IO15 is gone; now on net LED3: R29.1
Other:
- moved on the sheet: J10, Q7, Q8, R15, R28

Commit message: Milion błędów DRC do poprawienia
Connections:
- net ACC_IT1: now also U2.7 (IO35); no longer U2.6 (IO34)
- net ACC_IT2: now also U2.6 (IO34); no longer U2.7 (IO35)
- net AIN1: now also U2.12 (IO27); no longer U2.36 (IO22)
- net AIN2: now also U2.13 (IO14); no longer U2.37 (IO23)
- net BIN2: now also U2.10 (IO25); no longer U2.12 (IO27)
- net BOOT: no longer U1.19 (STBY), U4.19 (STBY)
- net CIN1: now also U2.31 (IO19); no longer U2.33 (IO21)
- net CIN2: now also U2.36 (IO22); no longer U2.10 (IO25)
- net DIN1: now also U2.37 (IO23); no longer U2.13 (IO14)
- net LIPO+: now also SW1.1 (A), SW1.6 (C); no longer SW1.2 (B), SW1.5 (B)
- net PWMA: now also R30.2, U2.14 (IO12); no longer U2.31 (IO19)
- net PWMB: now also U2.16 (IO13); no longer U2.30 (IO18)
- net PWMC: now also U2.33 (IO21); no longer R30.2, U2.14 (IO12)
- net PWMD: now also U2.30 (IO18); no longer U2.16 (IO13)
- net SW+: now also SW1.2 (B), SW1.5 (B); no longer SW1.1 (A), SW1.6 (C)
- net IO17 renamed STBY
- net STBY: now also U1.19 (STBY), U4.19 (STBY)
Changed lines of the file:
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@@
 	)
 	(junction
-		(at 201.93 120.65)
-		(diameter 0)
-		(color 0 0 0 0)
-	)
-	(junction
 		(at 336.55 92.71)
 		(diameter 0)
@@
 	(wire
 		(pts
-			(xy 209.55 115.57) (xy 201.93 115.57)
-		)
-		(stroke
-			(width 0)
-			(type default)
-		)
-	)
-	(wire
-		(pts
 			(xy 242.57 243.84) (xy 237.49 243.84)
 		)
@@
 	(wire
 		(pts
-			(xy 201.93 115.57) (xy 201.93 120.65)
-		)
-		(stroke
-			(width 0)
-			(type default)
-		)
-	)
-	(wire
-		(pts
 			(xy 316.23 109.22) (xy 318.77 109.22)
 		)
@@
 	(wire
 		(pts
-			(xy 193.04 120.65) (xy 201.93 120.65)
+			(xy 193.04 120.65) (xy 199.39 120.65)
 		)
 		(stroke
@@
 	(wire
 		(pts
-			(xy 243.84 69.85) (xy 248.92 69.85)
+			(xy 243.84 69.85) (xy 250.19 69.85)
 		)
 		(stroke
@@
 	(wire
 		(pts
-			(xy 201.93 120.65) (xy 209.55 120.65)
-		)
-		(stroke
-			(width 0)
-			(type default)
-		)
-	)
-	(wire
-		(pts
 			(xy 78.74 252.73) (xy 78.74 251.46)
 		)
@@
 	)
 	(rectangle
-		(start 224.79 26.67)
-		(end 401.32 78.74)
+		(start 222.25 26.67)
+		(end 398.78 78.74)
 		(stroke
 			(width 0)
@@
 		)
 	)
-	(label "PWMB"
-		(at 199.39 151.13 0)
+	(label "ACC_SCL"
+		(at 195.58 226.06 180)
 		(fields_autoplaced yes)
 		(effects
@@
 				(size 1.27 1.27)
 			)
-			(justify left bottom)
+			(justify right bottom)
 		)
 	)
-	(label "SW+"
-		(at 224.79 64.77 0)
+	(label "BIN1"
+		(at 199.39 166.37 0)
 		(fields_autoplaced yes)
 		(effects
@@
 		)
 	)
-	(label "ACC_SCL"
-		(at 195.58 226.06 180)
-		(fields_autoplaced yes)
-		(effects
-			(font
-				(size 1.27 1.27)
-			)
-			(justify right bottom)
-		)
-	)
 	(label "LED2"
 		(at 229.87 167.64 0)
@@
 		)
 	)
-	(label "IO17"
-		(at 199.39 148.59 0)
+	(label "SW+"
+		(at 250.19 69.85 0)
 		(fields_autoplaced yes)
 		(effects
@@
 		)
 	)
-	(label "PWMC"
-		(at 199.39 135.89 0)
+	(label "ACC_IT1"
+		(at 199.39 179.07 0)
 		(fields_autoplaced yes)
 		(effects
@@
 		)
 	)
-	(label "PWMA"
-		(at 199.39 153.67 0)
-		(fields_autoplaced yes)
-		(effects
-			(font
-				(size 1.27 1.27)
-			)
-			(justify left bottom)
-		)
-	)
 	(label "ACC_SDA"
 		(at 156.21 250.19 0)
@@
 		)
 	)
-	(label "AIN1"
-		(at 199.39 158.75 0)
-		(fields_autoplaced yes)
-		(effects
-			(font
-				(size 1.27 1.27)
-			)
-			(justify left bottom)
-		)
-	)
 	(label "SW+"
 		(at 358.14 53.34 0)
@@
 	)
 	(label "PWMC"
-		(at 210.82 154.94 0)
+		(at 199.39 156.21 0)
 		(fields_autoplaced yes)
 		(effects
@@
 		)
 	)
-	(label "ACC_IT2"
-		(at 199.39 179.07 0)
+	(label "CIN2"
+		(at 199.39 158.75 0)
 		(fields_autoplaced yes)
 		(effects
@@
 	)
 	(label "STBY"
-		(at 209.55 115.57 0)
+		(at 199.39 148.59 0)
 		(fields_autoplaced yes)
 		(effects
@@
 		)
 	)
-	(label "SW+"
+	(label "AIN2"
+		(at 199.39 140.97 0)
+		(fields_autoplaced yes)
+		(effects
+			(font
+				(size 1.27 1.27)
+			)
+			(justify left bottom)
+		)
+	)
+	(label "PWMD"
+		(at 199.39 151.13 0)
+		(fields_autoplaced yes)
+		(effects
+			(font
+				(size 1.27 1.27)
+			)
+			(justify left bottom)
+		)
+	)
+	(label "LIPO+"
 		(at 250.19 64.77 0)
 		(fields_autoplaced yes)
@@
 		)
 	)
+	(label "BIN2"
+		(at 199.39 163.83 0)
+		(fields_autoplaced yes)
+		(effects
+			(font
+				(size 1.27 1.27)
+			)
+			(justify left bottom)
+		)
+	)
 	(label "RX"
 		(at 43.18 100.33 0)
@@
 		)
 	)
+	(label "ACC_IT2"
+		(at 199.39 176.53 0)
+		(fields_autoplaced yes)
+		(effects
+			(font
+				(size 1.27 1.27)
+			)
+			(justify left bottom)
+		)
+	)
 	(label "PWMB"
 		(at 289.56 133.35 0)
@@
 		)
 	)
+	(label "CIN1"
+		(at 199.39 153.67 0)
+		(fields_autoplaced yes)
+		(effects
+			(font
+				(size 1.27 1.27)
+			)
+			(justify left bottom)
+		)
+	)
+	(label "LIPO+"
+		(at 224.79 64.77 0)
+		(fields_autoplaced yes)
+		(effects
+			(font
+				(size 1.27 1.27)
+			)
+			(justify left bottom)
+		)
+	)
 	(label "PWR+"
 		(at 350.52 165.1 0)
@@
 		)
 	)
-	(label "RTS"
-		(at 43.18 107.95 0)
+	(label "PWMA"
+		(at 210.82 154.94 0)
 		(fields_autoplaced yes)
 		(effects
@@
 		)
 	)
-	(label "ACC_SCL"
-		(at 199.39 130.81 0)
+	(label "PWMB"
+		(at 199.39 138.43 0)
 		(fields_autoplaced yes)
 		(effects
@@
 		)
 	)
-	(label "ACC_IT2"
-		(at 161.29 262.89 0)
+	(label "RTS"
+		(at 43.18 107.95 0)
 		(fields_autoplaced yes)
 		(effects
@@
 		)
 	)
-	(label "DIN1"
-		(at 199.39 140.97 0)
+	(label "ACC_SCL"
+		(at 199.39 130.81 0)
 		(fields_autoplaced yes)
 		(effects
@@
 		)
 	)
-	(label "LED4"
-		(at 78.74 228.6 0)
+	(label "ACC_IT2"
+		(at 161.29 262.89 0)
 		(fields_autoplaced yes)
 		(effects
@@
 		)
 	)
-	(label "BOOT"
-		(at 247.65 113.03 0)
+	(label "LED4"
+		(at 78.74 228.6 0)
 		(fields_autoplaced yes)
 		(effects
@@
 		)
 	)
-	(label "BIN2"
-		(at 199.39 168.91 0)
+	(label "BOOT"
+		(at 247.65 113.03 0)
 		(fields_autoplaced yes)
 		(effects
@@
 	)
 	(label "BOOT"
-		(at 209.55 120.65 0)
-		(fields_autoplaced yes)
-		(effects
-			(font
-				(size 1.27 1.27)
-			)
-			(justify left bottom)
-		)
-	)
-	(label "AIN2"
-		(at 199.39 161.29 0)
-		(fields_autoplaced yes)
-		(effects
-			(font
-				(size 1.27 1.27)
-			)
-			(justify left bottom)
-		)
-	)
-	(label "BIN1"
-		(at 199.39 166.37 0)
-		(fields_autoplaced yes)
-		(effects
-			(font
-				(size 1.27 1.27)
-			)
-			(justify left bottom)
-		)
-	)
-	(label "CIN2"
-		(at 199.39 163.83 0)
+		(at 199.39 120.65 0)
 		(fields_autoplaced yes)
 		(effects
@@
 		)
 	)
-	(label "LIPO+"
-		(at 224.79 69.85 0)
+	(label "DIN1"
+		(at 199.39 161.29 0)
 		(fields_autoplaced yes)
 		(effects
@@
 		)
 	)
-	(label "PWMD"
-		(at 199.39 138.43 0)
-		(fields_autoplaced yes)
-		(effects
-			(font
-				(size 1.27 1.27)
-			)
-			(justify left bottom)
-		)
-	)
 	(label "LED3"
 		(at 199.39 143.51 0)
@@
 		)
 	)
-	(label "ACC_IT1"
-		(at 199.39 176.53 0)
+	(label "BIN2"
+		(at 289.56 146.05 0)
 		(fields_autoplaced yes)
 		(effects
@@
 		)
 	)
-	(label "BIN2"
-		(at 289.56 146.05 0)
+	(label "AIN1"
+		(at 199.39 168.91 0)
 		(fields_autoplaced yes)
 		(effects
@@
 		)
 	)
-	(label "CIN1"
-		(at 199.39 156.21 0)
+	(label "PWR+"
+		(at 316.23 106.68 0)
 		(fields_autoplaced yes)
 		(effects
@@
 		)
 	)
-	(label "PWR+"
-		(at 316.23 106.68 0)
+	(label "BIN1"
+		(at 289.56 143.51 0)
 		(fields_autoplaced yes)
 		(effects
@@
 		)
 	)
-	(label "BIN1"
-		(at 289.56 143.51 0)
+	(label "SW+"
+		(at 224.79 69.85 0)
 		(fields_autoplaced yes)
 		(effects
@@
 		)
 	)
-	(label "LIPO+"
-		(at 248.92 69.85 0)
+	(label "PWMA"
+		(at 199.39 135.89 0)
 		(fields_autoplaced yes)
 		(effects

Commit message: prawie gotowe
Parts:
- removed C25: 100n, Capacitor_SMD:C_0603_1608Metric_Pad1.08x0.95mm_HandSolder, symbol Device:C
- added C26: 100n, Capacitor_SMD:C_0603_1608Metric_Pad1.08x0.95mm_HandSolder, symbol Device:C
- added R22: 10k, Resistor_SMD:R_0603_1608Metric_Pad0.98x0.95mm_HandSolder, symbol Device:R
- J6: footprint Connector_USB:USB_C_Receptacle_GCT_USB4110 -> Connector_USB:USB_C_Receptacle_GCT_USB4085
- SW2, SW3: footprint Button_Switch_SMD:SW_SPST_B3U-1000P -> Button_Switch_SMD:TSS 62 N
Connections:
- net +3.3V: now also R22.2
- net ACC_SCL: now also U2.27 (IO16); no longer U2.26 (IO4)
- net ACC_SDA: now also U2.26 (IO4); no longer U2.27 (IO16)
- net BOOT: now also U1.19 (STBY), C26.2, R22.1
- net CIN1: now also U2.33 (IO21); no longer U2.31 (IO19)
- net DIN1: now also U2.31 (IO19); no longer U2.37 (IO23)
- net GND: now also C26.1
- net LED4: now also U2.16 (IO13); no longer U2.9 (IO33)
- net LIPO+: no longer SW1.6 (C)
- net PWMB: now also U2.9 (IO33); no longer U2.16 (IO13)
- net PWMC: now also U2.37 (IO23); no longer U2.33 (IO21)
- net SW+: no longer SW1.5 (B)
- net STBY renamed STBY1
- net STBY1: no longer U1.19 (STBY)
- no-connect marks 7 -> 11
Other:
- note added: "Nie powinien być 0?"

Commit message: PRAWIE SKOŃCZONE
Parts:
- removed C15: 10n, Capacitor_SMD:C_0603_1608Metric_Pad1.08x0.95mm_HandSolder, symbol Device:C
- removed D8: GREEN, LED_SMD:LED_0805_2012Metric_Pad1.15x1.40mm_HandSolder, symbol Device:LED
- removed R26: 100, Resistor_SMD:R_0603_1608Metric_Pad0.98x0.95mm_HandSolder, symbol Device:R
- removed S1: AP22800HB-7, SON50P161X211X60-9N, symbol SamacSys_Parts:AP22800HB-7
- added C25: 100n, Capacitor_SMD:C_0603_1608Metric_Pad1.08x0.95mm_HandSolder, symbol Device:C
- added PS1: AP22814AW5-7, SOT95P285X130-5N, symbol SamacSys_Parts:AP22814AW5-7
- added TP1: TP_SDA, TestPoint:TestPoint_Pad_2.0x2.0mm, symbol Connector:Conn_01x01_Socket
- added TP10: TP_STBY1, TestPoint:TestPoint_Pad_2.0x2.0mm, symbol Connector:Conn_01x01_Socket
- added TP11: TP_PWMA_IO12, TestPoint:TestPoint_Pad_2.0x2.0mm, symbol Connector:Conn_01x01_Socket
- added TP12: TP_PWMB, TestPoint:TestPoint_Pad_2.0x2.0mm, symbol Connector:Conn_01x01_Socket
- added TP13: TP_AIN1, TestPoint:TestPoint_Pad_2.0x2.0mm, symbol Connector:Conn_01x01_Socket
- added TP14: TP_AIN2, TestPoint:TestPoint_Pad_2.0x2.0mm, symbol Connector:Conn_01x01_Socket
- added TP15: TP_BIN1, TestPoint:TestPoint_Pad_2.0x2.0mm, symbol Connector:Conn_01x01_Socket
- added TP16: TP_BIN2, TestPoint:TestPoint_Pad_2.0x2.0mm, symbol Connector:Conn_01x01_Socket
- added TP17: TP_STBY2, TestPoint:TestPoint_Pad_2.0x2.0mm, symbol Connector:Conn_01x01_Socket
- added TP18: TP_PWMC, TestPoint:TestPoint_Pad_2.0x2.0mm, symbol Connector:Conn_01x01_Socket
- added TP19: TP_PWMD, TestPoint:TestPoint_Pad_2.0x2.0mm, symbol Connector:Conn_01x01_Socket
- added TP2: TP_SCL, TestPoint:TestPoint_Pad_2.0x2.0mm, symbol Connector:Conn_01x01_Socket
- added TP20: TP_CIN1, TestPoint:TestPoint_Pad_2.0x2.0mm, symbol Connector:Conn_01x01_Socket
- added TP21: TP_CIN2, TestPoint:TestPoint_Pad_2.0x2.0mm, symbol Connector:Conn_01x01_Socket
- added TP22: TP_DIN1, TestPoint:TestPoint_Pad_2.0x2.0mm, symbol Connector:Conn_01x01_Socket
- added TP23: TP_DIN2, TestPoint:TestPoint_Pad_2.0x2.0mm, symbol Connector:Conn_01x01_Socket
- added TP4: TP_IO0, TestPoint:TestPoint_Pad_2.0x2.0mm, symbol Connector:Conn_01x01_Socket
- added TP5: TP_IO2, TestPoint:TestPoint_Pad_2.0x2.0mm, symbol Connector:Conn_01x01_Socket
- added TP6: TP_IO5, TestPoint:TestPoint_Pad_2.0x2.0mm, symbol Connector:Conn_01x01_Socket
- added TP7: TP_IO15, TestPoint:TestPoint_Pad_2.0x2.0mm, symbol Connector:Conn_01x01_Socket
- added TP8: TP_IT1, TestPoint:TestPoint_Pad_2.0x2.0mm, symbol Connector:Conn_01x01_Socket
- added TP9: TP_IT2, TestPoint:TestPoint_Pad_2.0x2.0mm, symbol Connector:Conn_01x01_Socket
- C14: value 10u -> 1u
- C16: value 1u -> 120u
- R27: value 1k -> 10k
Connections:
- net ACC_IT1: now also TP8.1 (Pin_1)
- net ACC_IT2: now also TP9.1 (Pin_1)
- net ACC_SCL: now also TP2.1 (Pin_1)
- net ACC_SDA: now also TP1.1 (Pin_1)
- net AIN1: now also TP13.1 (Pin_1)
- net AIN2: now also TP14.1 (Pin_1)
- net BIN1: now also TP15.1 (Pin_1)
- net BIN2: now also TP16.1 (Pin_1)
- net BOOT: now also TP17.1 (Pin_1), TP4.1 (Pin_1)
- net CIN1: now also TP20.1 (Pin_1)
- net CIN2: now also TP21.1 (Pin_1)
- net DIN1: now also TP22.1 (Pin_1)
- net DIN2: now also TP23.1 (Pin_1)
- net GND: now also C25.2, PS1.2 (GND)
- net LED1: now also TP5.1 (Pin_1)
- net LED2: now also TP6.1 (Pin_1)
- net LED3: now also TP7.1 (Pin_1)
- net LIPO+: now also R27.2, PS1.5 (IN)
- net PWMA: now also TP11.1 (Pin_1)
- net PWMB: now also TP12.1 (Pin_1)
- net PWMC: now also TP18.1 (Pin_1)
- net PWMD: now also TP19.1 (Pin_1)
- net PWR+: now also C25.1, PS1.1 (OUT); no longer R27.2
- net STBY1: now also TP10.1 (Pin_1)
- net SW+: now also PS1.4 (EN)
- net at R27.1: now also PS1.3 (FLG)
Other:
- moved on the sheet: C2, C3, IC4

Commit message: ZERO DRC ERRORS OMG OMG OMG
Parts:
- removed SW3: BOOT, Button_Switch_SMD:TSS 62 N, symbol Switch:SW_Push
- added SW3: BOOT, Button_Switch_SMD:TSS 62 N, symbol Switch:SW_Push_Dual
- added TP24: TP_3.3V, TestPoint:TestPoint_Pad_2.0x2.0mm, symbol Connector:Conn_01x01_Socket
- added TP3: TP_GND, TestPoint:TestPoint_Pad_2.0x2.0mm, symbol Connector:Conn_01x01_Socket
- C16: value 120u -> 100u; footprint Capacitor_SMD:C_0603_1608Metric_Pad1.08x0.95mm_HandSolder -> Capacitor_SMD:CP_Elec_5x5.3; symbol Device:C -> Device:C_Polarized
- R8: value 10k -> 0
- SW2: symbol Switch:SW_Push -> Switch:SW_Push_Dual
- TH1: symbol Device:Thermistor -> TermistorSMD:ThermistorSMD
Connections:
- net +3.3V: now also TP24.1 (Pin_1)
- net BOOT: now also SW3.3
- net EN: now also SW2.4; no longer SW2.2
- net GND: now also SW2.3, TP3.1 (Pin_1); no longer SW2.1
- net at R8.2: now also SW3.4
- no-connect marks 11 -> 15
Other:
- note removed: "Nie powinien być 0?"
- moved on the sheet: R8

Commit message: final commit2
Parts:
- AO1, AO2, BO1, BO2, CO1, CO2, DO1, DO2, TP1, TP10, TP11, TP12, TP13, TP14, TP15, TP16, TP17, TP18, TP19, TP2, TP20, TP21, TP22, TP23, TP24, TP3, TP4, TP5, TP6, TP7, TP8, TP9: now left out of the parts list
Changed lines of the file:
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@@
 		(unit 1)
 		(exclude_from_sim no)
-		(in_bom yes)
+		(in_bom no)
 		(on_board yes)
 		(dnp no)
@@
 		(unit 1)
 		(exclude_from_sim no)
-		(in_bom yes)
+		(in_bom no)
 		(on_board yes)
 		(dnp no)
@@
 		(unit 1)
 		(exclude_from_sim no)
-		(in_bom yes)
+		(in_bom no)
 		(on_board yes)
 		(dnp no)
@@
 		(unit 1)
 		(exclude_from_sim no)
-		(in_bom yes)
+		(in_bom no)
 		(on_board yes)
 		(dnp no)
@@
 		(unit 1)
 		(exclude_from_sim no)
-		(in_bom yes)
+		(in_bom no)
 		(on_board yes)
 		(dnp no)
@@
 		(unit 1)
 		(exclude_from_sim no)
-		(in_bom yes)
+		(in_bom no)
 		(on_board yes)
 		(dnp no)
@@
 		(unit 1)
 		(exclude_from_sim no)
-		(in_bom yes)
+		(in_bom no)
 		(on_board yes)
 		(dnp no)
@@
 		(unit 1)
 		(exclude_from_sim no)
-		(in_bom yes)
+		(in_bom no)
 		(on_board yes)
 		(dnp no)
@@
 		(unit 1)
 		(exclude_from_sim no)
-		(in_bom yes)
+		(in_bom no)
 		(on_board yes)
 		(dnp no)
@@
 		(unit 1)
 		(exclude_from_sim no)
-		(in_bom yes)
+		(in_bom no)
 		(on_board yes)
 		(dnp no)
@@
 		(unit 1)
 		(exclude_from_sim no)
-		(in_bom yes)
+		(in_bom no)
 		(on_board yes)
 		(dnp no)
@@
 		(unit 1)
 		(exclude_from_sim no)
-		(in_bom yes)
+		(in_bom no)
 		(on_board yes)
 		(dnp no)
@@
 		(unit 1)
 		(exclude_from_sim no)
-		(in_bom yes)
+		(in_bom no)
 		(on_board yes)
 		(dnp no)
@@
 		(unit 1)
 		(exclude_from_sim no)
-		(in_bom yes)
+		(in_bom no)
 		(on_board yes)
 		(dnp no)
@@
 		(unit 1)
 		(exclude_from_sim no)
-		(in_bom yes)
+		(in_bom no)
 		(on_board yes)
 		(dnp no)
@@
 		(unit 1)
 		(exclude_from_sim no)
-		(in_bom yes)
+		(in_bom no)
 		(on_board yes)
 		(dnp no)
@@
 		(unit 1)
 		(exclude_from_sim no)
-		(in_bom yes)
+		(in_bom no)
 		(on_board yes)
 		(dnp no)
@@
 		(unit 1)
 		(exclude_from_sim no)
-		(in_bom yes)
+		(in_bom no)
 		(on_board yes)
 		(dnp no)
@@
 		(unit 1)
 		(exclude_from_sim no)
-		(in_bom yes)
+		(in_bom no)
 		(on_board yes)
 		(dnp no)
@@
 		(unit 1)
 		(exclude_from_sim no)
-		(in_bom yes)
+		(in_bom no)
 		(on_board yes)
 		(dnp no)
@@
 		(unit 1)
 		(exclude_from_sim no)
-		(in_bom yes)
+		(in_bom no)
 		(on_board yes)
 		(dnp no)
@@
 		(unit 1)
 		(exclude_from_sim no)
-		(in_bom yes)
+		(in_bom no)
 		(on_board yes)
 		(dnp no)
@@
 		(unit 1)
 		(exclude_from_sim no)
-		(in_bom yes)
+		(in_bom no)
 		(on_board yes)
 		(dnp no)
@@
 		(unit 1)
 		(exclude_from_sim no)
-		(in_bom yes)
+		(in_bom no)
 		(on_board yes)
 		(dnp no)
@@
 		(unit 1)
 		(exclude_from_sim no)
-		(in_bom yes)
+		(in_bom no)
 		(on_board yes)
 		(dnp no)
@@
 		(unit 1)
 		(exclude_from_sim no)
-		(in_bom yes)
+		(in_bom no)
 		(on_board yes)
 		(dnp no)
@@
 		(unit 1)
 		(exclude_from_sim no)
-		(in_bom yes)
+		(in_bom no)
 		(on_board yes)
 		(dnp no)
@@
 		(unit 1)
 		(exclude_from_sim no)
-		(in_bom yes)
+		(in_bom no)
 		(on_board yes)
 		(dnp no)
@@
 		(unit 1)
 		(exclude_from_sim no)
-		(in_bom yes)
+		(in_bom no)
 		(on_board yes)
 		(dnp no)
@@
 		(unit 1)
 		(exclude_from_sim no)
-		(in_bom yes)
+		(in_bom no)
 		(on_board yes)
 		(dnp no)
@@
 		(unit 1)
 		(exclude_from_sim no)
-		(in_bom yes)
+		(in_bom no)
 		(on_board yes)
 		(dnp no)
@@
 		(unit 1)
 		(exclude_from_sim no)
-		(in_bom yes)
+		(in_bom no)
 		(on_board yes)
 		(dnp no)

Commit message: final commit5
Parts:
- removed J6: USB_C_Receptacle_PowerOnly_24P, Connector_USB:USB_C_Receptacle_GCT_USB4085, symbol Connector:USB_C_Receptacle_PowerOnly_24P
- removed R1, R2: 5.1k, Resistor_SMD:R_0603_1608Metric_Pad0.98x0.95mm_HandSolder, symbol Device:R
- added J1: 10118194-0001LF, 101181940001LF, symbol SamacSys_Parts:10118194-0001LF
- added R26, R32: 10k, Resistor_SMD:R_0603_1608Metric_Pad0.98x0.95mm_HandSolder, symbol Device:R
- D2: value LED -> GREEN
- D3: value LED -> RED
Connections:
- net GND: now also J1.4 (ID), J1.5 (GND), J1.MH1, J1.MH2, J1.MH3, J1.MH4, J1.MP1, J1.MP2, R26.1
- net VCC: now also J1.1 (VCC), R32.1
- new net: J1.2 (D-), R26.2
- new net: J1.3 (D+), R32.2
Other:
- moved on the sheet: C1, C14, C16, C2, C25, C3, C4, C5, D2, D3, IC1, IC4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
