File: projekt.kicad_pcb (KiCad board)
At the start: 4 copper layers, 65 x 65 mm, 93 parts, among them IC1 DW01+G, IC4 MIC5504-3.3YM5-TR, J10 Conn_01x06_Pin, J2 TP4056, J4 Conn_01x02_Socket, J6 USB_C_Receptacle_PowerOnly_24P, Q1 AO3400A, Q2 AO3400A, Q3 AO3400A, Q4 AO3400A, Q5 AO3400A, Q6 AO3400A, Q7 SS8050-HF, Q8 SS8050-HF, SW1 SW_Slide_DPDT, SW2 RST, SW3 BOOT, U1 TB6612FNG, U2 ESP32-WROOM-32E, U4 TB6612FNG

Commit message: Milion błędów DRC do poprawienia
Parts:
- moved D3 56.8 mm to (166.1, 70.4), turned to 0 degrees
- moved D2 56.5 mm to (166.1, 67.8), turned to 0 degrees
- moved SW1 56.4 mm to (122.8, 99.6), turned to -90 degrees
- moved R4 51.2 mm to (162.2, 70.4), turned to 180 degrees
- moved R3 51.1 mm to (162.3, 67.8), turned to 180 degrees
- moved C15 44.5 mm to (128.2, 102.2), turned to 0 degrees
- moved C14 44.1 mm to (127.3, 98.4), turned to -90 degrees
- moved D8 43.2 mm to (127.0, 107.4)
- moved R25 43.2 mm to (131.6, 107.4)
- moved S1 39.3 mm to (129.8, 100.1), turned to 0 degrees
- moved C16 38.9 mm to (129.9, 97.5), turned to 180 degrees
- moved R27 32.9 mm to (131.7, 103.8), turned to 0 degrees
- moved R26 32.8 mm to (133.2, 100.6), turned to 90 degrees
- moved DO2 32.6 mm to (123.4, 117.9), turned to -90 degrees
- moved AO1 30.3 mm to (175.3, 117.1), turned to 90 degrees
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Connections:
- R30 pad 2: /PWMC -> /PWMA
- SW1 pad 1: /SW+ -> /LIPO+
- SW1 pad 2: /LIPO+ -> /SW+
- SW1 pad 5: /LIPO+ -> /SW+
- SW1 pad 6: /SW+ -> /LIPO+
- U1 pad 19: /BOOT -> /STBY
- U2 pad 10: /CIN2 -> /BIN2
- U2 pad 12: /BIN2 -> /AIN1
- U2 pad 13: /DIN1 -> /AIN2
- U2 pad 14: /PWMC -> /PWMA
- U2 pad 16: /PWMD -> /PWMB
- U2 pad 28: /IO17 -> /STBY
- U2 pad 30: /PWMB -> /PWMD
- U2 pad 31: /PWMA -> /CIN1
- U2 pad 33: /CIN1 -> /PWMC
- U2 pad 36: /AIN1 -> /CIN2
- U2 pad 37: /AIN2 -> /DIN1
- U2 pad 6: /ACC_IT1 -> /ACC_IT2
- U2 pad 7: /ACC_IT2 -> /ACC_IT1
- U4 pad 19: /BOOT -> /STBY
Routing:
- net /STBY: track 0.00 -> 98.4 mm, vias 0 -> 3
- net /PWR+: track 32.5 -> 129.7 mm, vias 5 -> 24
- net /DIN1: track 0.00 -> 95.0 mm
- net /CIN2: track 0.00 -> 82.4 mm
- net /ACC_IT1: track 0.00 -> 60.0 mm, vias 0 -> 2
- net /ACC_IT2: track 0.00 -> 58.9 mm, vias 0 -> 2
- net /ACC_SDA: track 2.86 -> 61.2 mm
- net /ACC_SCL: track 3.85 -> 52.5 mm
- net /PWMC: track 2.98 -> 51.5 mm
- net /CIN1: track 0.00 -> 46.9 mm
- net /LED1: track 44.9 -> 91.1 mm, vias 2 -> 0
- net /DIN2: track 0.00 -> 45.7 mm, vias 0 -> 2
- net /PWMD: track 0.00 -> 41.7 mm
- net Net-(DO2-Pin_1): track 10.4 -> 49.4 mm, vias 0 -> 2
- net /BIN2: track 0.00 -> 38.6 mm
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- added copper zone on In1.Cu, net +3.3V
- added copper zone on B.Cu, net /LIPO+
- added copper zone on F.Cu, net /LIPO+
- added copper zone on In1.Cu, net /LIPO+
- added copper zone on B.Cu, net /LIPO-
- added copper zone on F.Cu, net /LIPO-
- added copper zone on B.Cu, net GND
- added copper zone on F.Cu, net GND
- added copper zone on In2.Cu, net GND
- removed copper zone on In2.Cu, net +3.3V

Commit message: prawie gotowe
Parts:
- removed C25: 100n, Capacitor_SMD:C_0603_1608Metric_Pad1.08x0.95mm_HandSolder
- added C26: 100n, Capacitor_SMD:C_0603_1608Metric_Pad1.08x0.95mm_HandSolder, F.Cu at (139.8, 104.5)
- added G***: LOGO, Graphics:small_logo, F.Cu at (163.1, 126.1)
- added G***: LOGO, Graphics:large_logo, B.Cu at (152.4, 95.0)
- added R22: 10k, Resistor_SMD:R_0603_1608Metric_Pad0.98x0.95mm_HandSolder, F.Cu at (141.5, 92.6)
- AO1, AO2, BO1, BO2, CO1, CO2, DO1, DO2: footprint TestPoint:TestPoint_Pad_2.0x2.0mm -> TestPoint:New TestPoint_Pad_2.0x2.0mm
- J6: footprint Connector_USB:USB_C_Receptacle_GCT_USB4110 -> Connector_USB:USB_C_Receptacle_GCT_USB4085
- SW2, SW3: footprint Button_Switch_SMD:SW_SPST_B3U-1000P -> Button_Switch_SMD:TSS 62 N
- moved C2 28.4 mm to (138.6, 88.2)
- moved IC4 28.2 mm to (141.8, 88.3)
- moved C3 27.9 mm to (145.1, 88.1)
- moved TH1 18.1 mm to (162.3, 93.2), turned to 180 degrees
- moved R6 14.5 mm to (162.4, 96.5), turned to 0 degrees
- moved SW2 7.95 mm to (169.5, 111.8), turned to -90 degrees
- moved R10 6.76 mm to (169.7, 119.3)
- moved R25 6.65 mm to (125.6, 104.5), turned to 90 degrees
- moved C1 6.61 mm to (156.5, 88.0)
- moved AO1 6.54 mm to (177.9, 111.1), turned to 0 degrees
- moved C4 6.16 mm to (149.6, 85.1)
- moved J2 6.11 mm to (151.4, 89.0)
- moved R5 5.78 mm to (155.1, 95.2), turned to 180 degrees
- moved C16 5.67 mm to (135.1, 99.8), turned to 0 degrees
- moved R7 5.61 mm to (156.8, 92.2), turned to 90 degrees
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Connections:
- SW1 pad 5: /SW+ -> unconnected-(SW1-B-Pad5)
- SW1 pad 6: /LIPO+ -> unconnected-(SW1-C-Pad6)
- U1 pad 19: /STBY -> /BOOT
- U2 pad 16: /PWMB -> /LED4
- U2 pad 26: /ACC_SCL -> /ACC_SDA
- U2 pad 27: /ACC_SDA -> /ACC_SCL
- U2 pad 28: /STBY -> /STBY1
- U2 pad 31: /CIN1 -> /DIN1
- U2 pad 33: /PWMC -> /CIN1
- U2 pad 37: /DIN1 -> /PWMC
- U2 pad 9: /LED4 -> /PWMB
- U4 pad 19: /STBY -> /STBY1
Routing:
- net GND: track 2.63 -> 165.7 mm, vias 13 -> 73
- net /STBY: track 98.4 -> 0.00 mm, vias 3 -> 0
- net /PWR+: track 129.7 -> 46.2 mm, vias 24 -> 27
- net VCC: track 107.9 -> 45.2 mm, vias 6 -> 12
- net /DIN1: track 95.0 -> 40.5 mm
- net /BOOT: track 34.5 -> 81.5 mm
- net /STBY1: track 0.00 -> 43.7 mm, vias 0 -> 2
- net /LED1: track 91.1 -> 54.1 mm, vias 0 -> 2
- net /DIN2: track 45.7 -> 80.8 mm, vias 2 -> 0
- net /CIN2: track 82.4 -> 51.1 mm
- net /LIPO+: track 23.6 -> 52.9 mm, vias 2 -> 11
- net /SW+: track 10.4 -> 34.4 mm, vias 0 -> 2
- net /ACC_SDA: track 61.2 -> 40.5 mm
- net +3.3V: track 44.9 -> 63.9 mm, vias 9 -> 11
- net /EN: track 50.4 -> 64.8 mm
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- added copper zone on In1.Cu, net VCC
- removed copper zone on B.Cu, net /LIPO+
- removed copper zone on B.Cu, net /LIPO-
- removed copper zone on F.Cu, net /LIPO-
- removed copper zone on B.Cu, net GND
- removed copper zone on F.Cu, net GND
Other:
- outline, holes or cut-outs redrawn
- board text added: "CONAN II"
- board text added: "Igor Santarek Kamil Lewiński 2024"

Commit message: PRAWIE SKOŃCZONE
Parts:
- removed C15: 10n, Capacitor_SMD:C_0603_1608Metric_Pad1.08x0.95mm_HandSolder
- removed D8: GREEN, LED_SMD:LED_0805_2012Metric_Pad1.15x1.40mm_HandSolder
- removed the G*** at (163.1, 126.1)
- removed the G*** at (152.4, 95.0)
- removed R26: 100, Resistor_SMD:R_0603_1608Metric_Pad0.98x0.95mm_HandSolder
- removed S1: AP22800HB-7, SamacSys_Parts:SON50P161X211X60-9N
- added C25: 100n, Capacitor_SMD:C_0603_1608Metric_Pad1.08x0.95mm_HandSolder, F.Cu at (131.7, 102.5)
- added G***: LOGO, Graphics:small_conan_logo, F.Cu at (163.4, 126.3)
- added PS1: AP22814AW5-7, SamacSys_Parts:SOT95P285X130-5N, F.Cu at (131.8, 99.1)
- added TP1: TP_SDA, TestPoint:TestPoint_Pad_2.0x2.0mm, F.Cu at (147.1, 78.5)
- added TP10: TP_STBY1, TestPoint:TestPoint_Pad_2.0x2.0mm, B.Cu at (166.1, 81.0)
- added TP11: TP_PWMA_IO12, TestPoint:TestPoint_Pad_2.0x2.0mm, B.Cu at (161.3, 66.5)
- added TP12: TP_PWMB, TestPoint:TestPoint_Pad_2.0x2.0mm, B.Cu at (180.2, 66.5)
- added TP13: TP_AIN1, TestPoint:TestPoint_Pad_2.0x2.0mm, B.Cu at (168.9, 66.5)
- added TP14: TP_AIN2, TestPoint:TestPoint_Pad_2.0x2.0mm, B.Cu at (165.1, 66.5)
- added TP15: TP_BIN1, TestPoint:TestPoint_Pad_2.0x2.0mm, B.Cu at (172.7, 66.5)
- added TP16: TP_BIN2, TestPoint:TestPoint_Pad_2.0x2.0mm, B.Cu at (176.4, 66.5)
- added TP17: TP_STBY2, TestPoint:TestPoint_Pad_2.0x2.0mm, B.Cu at (131.1, 76.8)
- added TP18: TP_PWMC, TestPoint:TestPoint_Pad_2.0x2.0mm, B.Cu at (125.6, 66.7)
- added TP19: TP_PWMD, TestPoint:TestPoint_Pad_2.0x2.0mm, B.Cu at (141.2, 66.7)
- added TP2: TP_SCL, TestPoint:TestPoint_Pad_2.0x2.0mm, F.Cu at (151.1, 79.1)
- added TP20: TP_CIN1, TestPoint:TestPoint_Pad_2.0x2.0mm, B.Cu at (133.5, 66.7)
- added TP21: TP_CIN2, TestPoint:TestPoint_Pad_2.0x2.0mm, B.Cu at (129.5, 66.7)
- added TP22: TP_DIN1, TestPoint:TestPoint_Pad_2.0x2.0mm, B.Cu at (137.5, 66.7)
- added TP23: TP_DIN2, TestPoint:TestPoint_Pad_2.0x2.0mm, B.Cu at (144.9, 66.7)
- added TP4: TP_IO0, TestPoint:TestPoint_Pad_2.0x2.0mm, F.Cu at (125.7, 107.2)
- added TP5: TP_IO2, TestPoint:TestPoint_Pad_2.0x2.0mm, F.Cu at (163.7, 112.0)
- added TP6: TP_IO5, TestPoint:TestPoint_Pad_2.0x2.0mm, F.Cu at (127.6, 119.8)
- added TP7: TP_IO15, TestPoint:TestPoint_Pad_2.0x2.0mm, F.Cu at (174.8, 119.5)
- added TP8: TP_IT1, TestPoint:TestPoint_Pad_2.0x2.0mm, F.Cu at (141.2, 66.7)
- added TP9: TP_IT2, TestPoint:TestPoint_Pad_2.0x2.0mm, F.Cu at (137.5, 66.7)
- AO1, AO2, BO1, BO2, CO1, CO2, DO1, DO2: footprint TestPoint:New TestPoint_Pad_2.0x2.0mm -> TestPoint:TestPoint_Pad_2.0x2.0mm
- C14: value 10u -> 1u
- C16: value 1u -> 120u
- R27: value 1k -> 10k
- moved R1 11.0 mm to (179.0, 90.7), turned to 180 degrees
- moved C16 6.65 mm to (128.7, 101.3), turned to -90 degrees
- moved AO2 6.22 mm to (177.9, 109.7)
- moved R2 5.43 mm to (174.6, 99.2)
- moved R27 5.21 mm to (135.8, 99.4), turned to 90 degrees
- moved R25 5.07 mm to (130.3, 106.4), turned to 180 degrees
- moved AO1 4.82 mm to (176.4, 115.7)
- moved CO2 3.71 mm to (122.2, 78.1)
- moved J6 3.47 mm to (177.2, 100.0)
- moved C14 2.50 mm to (131.7, 95.6)
- moved CO1 0.97 mm to (124.7, 74.9)
- moved C5 0.46 mm to (132.0, 85.4)
- moved C21 0.38 mm to (163.8, 76.1)
- moved C9 0.25 mm to (136.7, 83.2)
- moved C19 0.15 mm to (163.7, 87.4)
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Connections:
- R27 pad 2: /PWR+ -> /LIPO+
Routing:
- net /AIN2: track 27.8 -> 72.4 mm, vias 0 -> 1
- net /PWMB: track 38.3 -> 81.6 mm, vias 0 -> 1
- net /AIN1: track 29.8 -> 72.5 mm, vias 0 -> 1
- net /PWMA: track 28.5 -> 70.7 mm, vias 0 -> 1
- net /BIN1: track 33.6 -> 74.8 mm, vias 0 -> 1
- net /BIN2: track 35.9 -> 76.4 mm, vias 0 -> 1
- net GND: track 165.7 -> 128.2 mm, vias 73 -> 60
- net Net-(AO2-Pin_1): track 48.6 -> 11.5 mm, vias 6 -> 4
- net Net-(DO2-Pin_1): track 50.6 -> 14.1 mm, vias 6 -> 4
- net Net-(DO1-Pin_1): track 42.5 -> 11.2 mm, vias 6 -> 4
- net Net-(AO1-Pin_1): track 41.5 -> 12.1 mm, vias 6 -> 4
- net /LED1: track 54.1 -> 81.8 mm, vias 2 -> 4
- net /ACC_IT2: track 62.8 -> 79.0 mm, vias 0 -> 2
- net /PWMD: track 38.0 -> 54.1 mm, vias 0 -> 1
- net /DIN1: track 40.5 -> 55.9 mm, vias 0 -> 1
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- added copper zone on B.Cu, net Net-(AO1-Pin_1)
- added copper zone on B.Cu, net Net-(AO2-Pin_1)
- added copper zone on B.Cu, net Net-(DO1-Pin_1)
- added copper zone on B.Cu, net Net-(DO2-Pin_1)
- removed copper zone on F.Cu, net /PWR+
Other:
- outline, holes or cut-outs redrawn
